File: V0.0/Apple2Card.kicad_pcb (KiCad board)
At the start: 2 copper layers, 213.5 x 79.1 mm, 62 parts, among them J1 Conn_01x08_Pin, P2 Conn_02x13_Top_Bottom, SW1 SW_DIP_x08, U1C1 74LS240, U1E1 74LS14, U2 74LS133, U2B1 74LS08, U2D1 74LS138, U2E1 74LS09, U3A1 2764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

Commit message: menage
Connections:
- U3C1 pad 8: Net-(U3C1-I7) -> Net-(U3C1-I8)
- U4E1 pad 1: Net-(U4E1-A->B) -> Net-(U3C1-I7)
- U5E1 pad 4: Net-(U4E1-A->B) -> Net-(U3C1-I7)
- U6C1 pad 4: Net-(U3C1-I7) -> Net-(U3C1-I8)
- U6C1 pad 5: Net-(U4E1-A->B) -> Net-(U3C1-I7)
- U6E1 pad 9: Net-(U3C1-I7) -> Net-(U3C1-I8)
Routing:
- net Net-(U3C1-I8): track 0.00 -> 120.3 mm, vias 0 -> 1
- net Net-(U4E1-A->B): track 113.7 -> 0.00 mm, vias 3 -> 0
- net Net-(U3C1-I7): track 138.7 -> 151.1 mm, vias 1 -> 5
- net Net-(U3C1-IO1): track 165.4 -> 166.0 mm
Other:
- board text added: "10/04/2026"
- board text added: "Rev B."
- board text removed: "29/03/2026"
